Commit message: feat: Add agent47 integration for networked agents
- Update CMakeLists.txt to ignore -Wno-maybe-uninitialized and -Wno-unused-function warnings.
- Update agent47 dependency to 0.0.14.
- Add GNSS, IMU, and LIDAR sensors to example URDFs (husky, oxbo_harvester, tractor, trailer).
- Refactor agent to use agent47 PipeBridge for networked communication, removing custom RPC peer.
- Remove `teleport` method from Agent as it's not supported by agent47 comms yet.
- Remove `set_teleport_callback` from Agent.
- Remove flatsim::RpcPeer dependencies from agent.hpp.
- Introduce netpipe::Pipe and agent47::PipeBridge for simulator-agent communication.
- Remove flatsim::RpcPeer from simulator.hpp.
- Implement `process_agent47_connections` in Simulator for new agent47 peer connections.
- Implement `cleanup_stale_connections` for agent47 peers.
- Implement `register_agent47_handlers`, including `AGENT47_METHOD_COMMAND`, `AGENT47_METHOD_HEARTBEAT`, and `AGENT47_METHOD_MODEL`.
- Implement `serialize_agent47_feedback` and `serialize_agent47_sensor` for agent47 protocol.
- Implement `apply_agent47_command` to translate agent47 commands to machine controls.
- Implement `bind_agent47_peer_to_uuid` to manage agent UUIDs during model loading.
- Update `machine_from_model` to parse LIDAR configuration from URDF sensor properties.
- Remove direct `teleport_callback_` usage in Simulator.
- Replace `spawn_requests` with `agent47_connections` in simulator loop.

File: examples/machines/urdf/husky.urdf (robot description, URDF)
Before this commit: robot husky, 8 links, 7 joints
Links:
- added link gnss_link
- added link imu_link
- added link lidar_link
- added link sensor_link
Joints:
- added joint gnss_joint: type fixed, parent sensor_link, child gnss_link, origin xyz=0 0 0 rpy=0 0 0
- added joint imu_joint: type fixed, parent sensor_link, child imu_link, origin xyz=0 0 0 rpy=0 0 0
- added joint lidar_joint: type fixed, parent sensor_link, child lidar_link, origin xyz=0 0 0 rpy=0 0 0
- added joint sensor_joint: type fixed, parent base_link, child sensor_link, origin xyz=0 0 0 rpy=0 0 0

File: examples/machines/urdf/oxbo_harvester.urdf (robot description, URDF)
Before this commit: robot harvester, 17 links, 16 joints
Links:
- added link gnss_link
- added link imu_link
- added link lidar_link
- added link sensor_link
Joints:
- added joint gnss_joint: type fixed, parent sensor_link, child gnss_link, origin xyz=0 0 0 rpy=0 0 0
- added joint imu_joint: type fixed, parent sensor_link, child imu_link, origin xyz=0 0 0 rpy=0 0 0
- added joint lidar_joint: type fixed, parent sensor_link, child lidar_link, origin xyz=0 0 0 rpy=0 0 0
- added joint sensor_joint: type fixed, parent base_link, child sensor_link, origin xyz=0 0 0 rpy=0 0 0

File: examples/machines/urdf/tractor.urdf (robot description, URDF)
Before this commit: robot tractor, 13 links, 12 joints
Links:
- added link gnss_link
- added link imu_link
- added link lidar_link
- added link sensor_link
Joints:
- added joint gnss_joint: type fixed, parent sensor_link, child gnss_link, origin xyz=0 0 0 rpy=0 0 0
- added joint imu_joint: type fixed, parent sensor_link, child imu_link, origin xyz=0 0 0 rpy=0 0 0
- added joint lidar_joint: type fixed, parent sensor_link, child lidar_link, origin xyz=0 0 0 rpy=0 0 0
- added joint sensor_joint: type fixed, parent base_link, child sensor_link, origin xyz=0 0 0 rpy=0 0 0

File: examples/machines/urdf/trailer.urdf (robot description, URDF)
Before this commit: robot trailer, 10 links, 9 joints
Links:
- added link gnss_link
- added link imu_link
- added link lidar_link
- added link sensor_link
Joints:
- added joint gnss_joint: type fixed, parent sensor_link, child gnss_link, origin xyz=0 0 0 rpy=0 0 0
- added joint imu_joint: type fixed, parent sensor_link, child imu_link, origin xyz=0 0 0 rpy=0 0 0
- added joint lidar_joint: type fixed, parent sensor_link, child lidar_link, origin xyz=0 0 0 rpy=0 0 0
- added joint sensor_joint: type fixed, parent base_link, child sensor_link, origin xyz=0 0 0 rpy=0 0 0
